File: Dive_Computer.kicad_sch (KiCad schematic)
At the start: 24 parts, among them IC1 LTC4120EUD-4.2#PBF, IC2 MS583730BA01-50, U1 ESP32-C3_SUPERMINI_TH

Commit message: Schematic finished
Parts:
- added J1: SCREEN, Connector_Hirose:Hirose_DF13-07P-1.25DSA_1x07_P1.25mm_Vertical, symbol Connector:Conn_01x07_Socket
- added JP1: SolderJumper_2_Open, symbol Jumper:SolderJumper_2_Open
- added R6, R7, R8, R9: 10k, Resistor_SMD:R_0603_1608Metric, symbol Device:R_Small
- BATTERIE1: renamed from BATTERIE; footprint (none) -> Connector_Hirose:Hirose_DF13-02P-1.25DSA_1x02_P1.25mm_Vertical
- IC1: footprint QFN50P300X300X80-17N-D -> Package_DFN_QFN:QFN-16-1EP_3x3mm_P0.5mm_EP1.7x1.7mm
- IC2: footprint MS583730BA0150 -> Sensor_Pressure:TE_MS5837-xxBA
- R1, R2, R3, R4, R5: footprint (none) -> Resistor_SMD:R_0603_1608Metric
Connections:
- net +3.3V: now also U1.3.3 (3V3), R8.2, R9.2
- net BAT+: now also J1.2 (Pin_2), R6.2
- net GND: now also J1.1 (Pin_1), R7.1
- net SCL: now also U1.9 (GPIO9)
- net SDA: now also U1.8 (GPIO8)
- net ~{CHRG}: now reaches IC1.14 (~{CHRG})
- net ~{CHRG}: now also U1.20 (GPIO20), R8.1
- net ~{FLT}: now reaches IC1.15 (~{FAULT})
- net ~{FLT}: now also JP1.2 (B), R9.1
- net INT2: now reaches LIS12DUX1.11 (INT2)
- net INT2: now also U1.1 (GPIO1)
- net INT1: now reaches LIS12DUX1.12 (INT1)
- net INT1: now also U1.0 (GPIO0)
- net Data/Command: now reaches U1.10 (GPIO10)
- net Data/Command: now also J1.3 (Pin_3)
- net at U1.21 (GPIO21): now also JP1.1 (A)
- net at U1.3 (GPIO3): now also R6.1, R7.2
- net SPI_CLK: now reaches U1.4 (GPIO4)
- net SPI_CLK: now also J1.4 (Pin_4)
- net MISO: now reaches U1.5 (GPIO5)
- net MISO: now also J1.6 (Pin_6)
- net MOSI: now reaches U1.6 (GPIO6)
- net MOSI: now also J1.7 (Pin_7)
- net CS: now reaches U1.7 (GPIO7)
- net CS: now also J1.5 (Pin_5)
- no-connect marks 0 -> 1
Other:
- moved on the sheet: C3, R4, R5

Commit message: Schematic update
Parts:
- added C10, C9: 100n, Capacitor_SMD:C_0603_1608Metric, symbol Device:C_Small
- added Q1: Si2301HDS, Package_TO_SOT_SMD:TSOT-23, symbol Simulation_SPICE:PMOS
- added R10: 10k, Resistor_SMD:R_0603_1608Metric, symbol Device:R_Small
- added U2: Si7201-03-IV, Package_TO_SOT_SMD:SOT-23, symbol Sensor_Magnetic:A1102xLH
- C1, C3, C6: footprint (none) -> Capacitor_SMD:C_1210_3225Metric
- C2, C4, C5, C7, C8: footprint (none) -> Capacitor_SMD:C_0603_1608Metric
- D1, D2, D3, D4: footprint (none) -> Diode_SMD:D_MicroSMP_LargeCathode
- JP1: footprint (none) -> Jumper:SolderJumper-2_P1.3mm_Open_RoundedPad1.0x1.5mm
- L1: footprint (none) -> Inductor_SMD:L_APV_ANR4018
- Power_Inductor1: footprint Inductor_THT_Wurth:L_Wurth_WE-WPCC-RX_760308101303 -> Connector_PinHeader_2.54mm:PinHeader_1x02_P2.54mm_Vertical
Connections:
- net +3.3V: now also C10.2
- net BAT+: now also C9.2, Q1.3 (S), R10.1, U2.1 (V_{CC}); no longer C6.1, D4.2 (A), IC1.10 (BATSNS), IC1.9 (BAT)
- net GND: now also C10.1, C9.1, U2.3 (GND)
- new net: Q1.2 (G), R10.2, U2.2 (V_{OUT})
- new net VCC: C6.1, D4.2 (A), IC1.10 (BATSNS), IC1.9 (BAT), Q1.1 (D)
Other:
- note added: "Freedinving Computer"
- moved on the sheet: D4, JP1, R6, R7, U1

Commit message: Routage terminé
Parts:
- C1, C6: footprint Capacitor_SMD:C_1210_3225Metric -> Capacitor_SMD:C_0603_1608Metric
Connections:
- net BAT+: no longer J1.2 (Pin_2), R6.2
- net VCC: now also J1.2 (Pin_2), R6.2
- net at C3.1, IC1.16 (RUN), R4.1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: no longer D2.1 (K), D3.1 (K), IC1.3 (IN), R4.2
- new net: D2.1 (K), D3.1 (K), IC1.3 (IN), R4.2
Changed lines of the file:
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@@
 	)
 	(junction
-		(at 60.96 39.37)
-		(diameter 0)
-		(color 0 0 0 0)
-	)
-	(junction
 		(at 259.08 90.17)
 		(diameter 0)
@@
 	)
 	(junction
-		(at 60.96 43.18)
-		(diameter 0)
-		(color 0 0 0 0)
-	)
-	(junction
 		(at 251.46 90.17)
 		(diameter 0)
@@
 	(wire
 		(pts
-			(xy 60.96 39.37) (xy 66.04 39.37)
-		)
-		(stroke
-			(width 0)
-			(type default)
-		)
-	)
-	(wire
-		(pts
 			(xy 48.26 41.91) (xy 48.26 39.37)
 		)
@@
 	(wire
 		(pts
-			(xy 59.69 39.37) (xy 60.96 39.37)
+			(xy 59.69 39.37) (xy 66.04 39.37)
 		)
 		(stroke
@@
 	(wire
 		(pts
-			(xy 220.98 57.15) (xy 237.49 57.15)
+			(xy 220.98 57.15) (xy 231.14 57.15)
 		)
 		(stroke
@@
 	(wire
 		(pts
-			(xy 60.96 39.37) (xy 60.96 43.18)
-		)
-		(stroke
-			(width 0)
-			(type default)
-		)
-	)
-	(wire
-		(pts
 			(xy 217.17 85.09) (xy 217.17 87.63)
 		)
@@
 		)
 	)
-	(label "BAT+"
-		(at 22.86 104.14 270)
-		(effects
-			(font
-				(size 1.27 1.27)
-			)
-			(justify right bottom)
-		)
-	)
 	(label "CS"
 		(at 91.44 107.95 180)
@@
 		)
 	)
-	(label "BAT+"
-		(at 237.49 57.15 180)
-		(effects
-			(font
-				(size 1.27 1.27)
-			)
-			(justify right bottom)
-		)
-	)
 	(label "Data{slash}Command"
 		(at 91.44 115.57 180)
@@
 	)
 	(symbol
+		(lib_id "power:VCC")
+		(at 231.14 57.15 270)
+		(unit 1)
+		(body_style 1)
+		(exclude_from_sim no)
+		(in_bom yes)
+		(on_board yes)
+		(in_pos_files yes)
+		(dnp no)
+		(fields_autoplaced yes)
+		(property "Reference" "#PWR023"
+			(at 227.33 57.15 0)
+			(hide yes)
+			(show_name no)
+			(do_not_autoplace no)
+			(effects
+				(font
+					(size 1.27 1.27)
+				)
+			)
+		)
+		(property "Value" "VCC"
+			(at 234.95 57.1499 90)
+			(show_name no)
+			(do_not_autoplace no)
+			(effects
+				(font
+					(size 1.27 1.27)
+				)
+				(justify left)
+			)
+		)
+		(property "Footprint" ""
+			(at 231.14 57.15 0)
+			(hide yes)
+			(show_name no)
+			(do_not_autoplace no)
+			(effects
+				(font
+					(size 1.27 1.27)
+				)
+			)
+		)
+		(property "Datasheet" ""
+			(at 231.14 57.15 0)
+			(hide yes)
+			(show_name no)
+			(do_not_autoplace no)
+			(effects
+				(font
+					(size 1.27 1.27)
+				)
+			)
+		)
+		(property "Description" "Power symbol creates a global label with name \"VCC\""
+			(at 231.14 57.15 0)
+			(hide yes)
+			(show_name no)
+			(do_not_autoplace no)
+			(effects
+				(font
+					(size 1.27 1.27)
+				)
+			)
+		)
+		(pin "1"
+		)
+		(instances
+			(project "Dive_Computer"
+				(path "/6749645a-a7ea-4eb0-9e4c-e6953362916c"
+					(reference "#PWR023")
+					(unit 1)
+				)
+			)
+		)
+	)
+	(symbol
 		(lib_id "power:+3.3V")
 		(at 82.55 102.87 270)
@@
 			)
 		)
-		(property "Footprint" "Capacitor_SMD:C_1210_3225Metric"
+		(property "Footprint" "Capacitor_SMD:C_0603_1608Metric"
 			(at 116.84 63.5 0)
 			(hide yes)
@@
 			)
 		)
-		(property "Footprint" "Capacitor_SMD:C_1210_3225Metric"
+		(property "Footprint" "Capacitor_SMD:C_0603_1608Metric"
 			(at 259.08 85.09 0)
 			(hide yes)
@@
 					(unit 1)
 				)
+			)
+		)
+	)
+	(symbol
+		(lib_id "power:VCC")
+		(at 22.86 104.14 0)
+		(unit 1)
+		(body_style 1)
+		(exclude_from_sim no)
+		(in_bom yes)
+		(on_board yes)
+		(in_pos_files yes)
+		(dnp no)
+		(fields_autoplaced yes)
+		(property "Reference" "#PWR022"
+			(at 22.86 107.95 0)
+			(hide yes)
+			(show_name no)
+			(do_not_autoplace no)
+			(effects
+				(font
+					(size 1.27 1.27)
+				)
+			)
+		)
+		(property "Value" "VCC"
+			(at 22.86 99.06 0)
+			(show_name no)
+			(do_not_autoplace no)
+			(effects
+				(font
+					(size 1.27 1.27)
+				)
+			)
+		)
+		(property "Footprint" ""
+			(at 22.86 104.14 0)
+			(hide yes)
+			(show_name no)
+			(do_not_autoplace no)
+			(effects
+				(font
+					(size 1.27 1.27)
+				)
+			)
+		)
+		(property "Datasheet" ""
+			(at 22.86 104.14 0)
+			(hide yes)
+			(show_name no)
+			(do_not_autoplace no)
+			(effects
+				(font
+					(size 1.27 1.27)
+				)
+			)
+		)
+		(property "Description" "Power symbol creates a global label with name \"VCC\""
+			(at 22.86 104.14 0)
+			(hide yes)
+			(show_name no)
+			(do_not_autoplace no)
+			(effects
+				(font
+					(size 1.27 1.27)
+				)
+			)
+		)
+		(pin "1"
+		)
+		(instances
+			(project "Dive_Computer"
+				(path "/6749645a-a7ea-4eb0-9e4c-e6953362916c"
+					(reference "#PWR022")
+					(unit 1)
+				)
