File: Hardware/V1/Charger/Chargeur/Chargeur.kicad_sch (KiCad schematic)
At the start: 30 parts, among them J1 USB_C_Receptacle_PowerOnly_6P, U1 LTC4125

Commit message: Ibom charger
Parts:
- added C9: 1u, Capacitor_SMD:C_1206_3216Metric, symbol Device:C_Small
- added H1, H2: MountingHole_Pad, MountingHole:MountingHole_3.2mm_M3_DIN965_Pad, symbol Mechanical:MountingHole_Pad
- C7, C8: footprint Capacitor_SMD:C_0603_1608Metric -> Capacitor_SMD:C_1206_3216Metric
Connections:
- net +5V: now also C9.1
- net GND: now also C9.2
