File: Hardware/V2/DiveComputerV2/DiveComputerV2.kicad_sch (KiCad schematic)
At the start: 7 parts, among them IC2 MS583730BA01-50, U1 STM32L4P5CEU6, U2 LIS2DW12TR

Commit message: added magnetometer & haptic driver
Parts:
- added U3: TLI493DA2B6HTSA1, easyeda2kicad:TSOP-6_L3.0-W1.5-P0.95-LS2.8-BR, symbol easyeda2kicad:TLI493DA2B6HTSA1
- added U4: DRV2624YFFR, easyeda2kicad:DSBGA-9_L1.4-W1.3-R3-C3-P0.40-BL, symbol easyeda2kicad:DRV2624YFFR
- LIS2DW12TR: renamed from LIS12DUX1; LCSC Part (none) -> C189624
Other:
- note added: "HAPTIC DRIVER"
- note added: "MAGNETOMETER"
- note added: "STM32"
- note added: "To add: -haptic motor -nfc comm & charging -screen connector -jtag"
- note removed: "To add: -hall sensor -haptic motor & driver -nfc comm & charging -screen connector -jtag"
- moved on the sheet: C1, C2, LIS2DW12TR, U2
