File: V2/Hardware/DiveComputerV2/DiveComputerV2.kicad_sch (KiCad schematic)
At the start: 86 parts, among them J1 Conn_01x01_Socket, J2 Conn_01x01_Socket, J3 Conn_01x02_Socket, U1 LIS2MDL, U10 MS583730BA01-50, U11 TPS7A0331PDQNR, U12 TPS75105DSKR, U2 NRF52833-QDAA-R, U3 TPS7A0218PDQNR, U4 DRV2624YFFR, U5 BQ51051BRHLR, U6 TPS7A0212PYCHR, U8 VEML6035, U9 TMAG3001A1Y, X1 ECS-320-CDX-2152, X2 CM8V-T1A-32.768KHZ-9PF-20PPM-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

Commit message: PCB layout
Parts:
- removed C25, C27, C28, C29, C48, C49: 1u, Capacitor_SMD:C_0402_1005Metric, symbol Device:C_Small
- removed C31: 4.7u, Capacitor_SMD:C_0402_1005Metric, symbol Device:C_Small
- removed C39: 100p, Capacitor_SMD:C_0402_1005Metric, symbol Device:C_Small
- removed C42: 12p, Capacitor_SMD:C_0402_1005Metric, symbol Device:C_Small
- added C11, C12, C26: 12p, Capacitor_SMD:C_0402_1005Metric, symbol Device:C_Small
- added C14: 4.7u, Capacitor_SMD:C_0402_1005Metric, symbol Device:C_Small
- added C15, C34, C35, C43: 1u, Capacitor_SMD:C_0402_1005Metric, symbol Device:C_Small
- added C22: 100p, Capacitor_SMD:C_0402_1005Metric, symbol Device:C_Small
- added R3: 22k, Resistor_SMD:R_0402_1005Metric, symbol Device:R_Small
- C13: renamed from C32; LCSC Part C368809 -> C23733; MPN CL05A475KP5NRNC -> (none)
- C21: renamed from C50; LCSC Part C281751 -> C1546; MPN CC0402KRX7R9BB101 -> 0402CG101J500NT
- C25: renamed from C43; LCSC Part C526985 -> C1547; MPN CC0402GRNPO9BN120 -> 0402CG120J500NT
- C36: LCSC Part C29266 -> C52923; MPN CL05A105KO5NNNC -> CL05A105KA5NQNC
- C44, C45: value 12p -> 1u; LCSC Part C526985 -> C52923; MPN CC0402GRNPO9BN120 -> CL05A105KA5NQNC
- C46: renamed from C16; LCSC Part C29266 -> C52923; MPN CL05A105KO5NNNC -> CL05A105KA5NQNC
- C7: renamed from C1; LCSC Part C315248 -> C15525; MPN CL05A106MP5NUNC -> (none)
- C8: renamed from C23; LCSC Part C315248 -> C15525; MPN CL05A106MP5NUNC -> (none)
- R4: renamed from R10; value 26.7k -> 4.7k; LCSC Part C324918 -> C25900; MPN RC-02K2672FT -> 0402WGF4701TCE
- R7: renamed from R12; LCSC Part C60485 -> C17168; MPN RC0402JR-070RL -> (none)
- R8: renamed from R11; LCSC Part C60485 -> C17168; MPN RC0402JR-070RL -> (none)
- R9: renamed from R7; LCSC Part C60485 -> C17168; MPN RC0402JR-070RL -> (none)
- renumbered C4 to C1, C2 to C10, C33 to C16, C37 to C17, C38 to C18, C34 to C19, C10 to C2, C35 to C20, C40 to C23, C41 to C24, C46 to C27, C47 to C28, C6 to C29, C21 to C3, C18 to C31, C12 to C32, C11 to C33, C7 to C37, C8 to C38, C9 to C39, C26 to C4, C13 to C40, C14 to C41, C15 to C42, C20 to C47, C17 to C48, C22 to C49, C3 to C5, C5 to C6, C24 to C9, L3 to L1, L4 to L3, L5 to L4, L1 to L5, LIS2DUX12 to LIS2DUX1, R9 to R1, R5 to R10, R6 to R11, R3 to R12, R4 to R13, R8 to R2, R1 to R5, R2 to R6, U3 to U10, U5 to U11, U8 to U2, U4 to U3, U9 to U4, U10 to U5, U12 to U6, U2 to U7, U6 to U8, U11 to U9, X2 to X1, X1 to X2
Connections:
- net +1.2V: now also FPC1.15, FPC1.16, FPC1.18, FPC1.19, C34.2; no longer FPC1.5, FPC1.6, FPC1.8, FPC1.9
- net +1.8V: now also C36.2, FPC1.11, FPC1.21; no longer FPC1.13, FPC1.3
- net +3.1V: now also FPC1.22, C35.2; no longer FPC1.2
- net BAT+: now also C44.2, C45.2, C14.1, C43.2
- net BL: now also FPC1.2; no longer FPC1.22
- net GND: now also C44.1, C45.1, FPC1.1, FPC1.14, FPC1.20, FPC1.6, FPC1.9, C11.2, C12.2, C14.2, C15.1, C22.1, C26.1, C34.1, C35.1, C43.1, R3.2; no longer C44.2, C45.2, FPC1.10, FPC1.15, FPC1.18, FPC1.23, FPC1.4, R4.2
- net OUT+: now also J2.1 (Pin_1); no longer J1.1 (Pin_1)
- net OUT-: now also J1.1 (Pin_1); no longer J2.1 (Pin_1)
- net SCREEN_SDI: now also FPC1.13; no longer FPC1.11
- net SCREEN_~{CS}: now also FPC1.10; no longer FPC1.14
- net SCREEN_~{RST}: now also FPC1.8; no longer FPC1.16
- net SWDCLK: now also C29.4 (SWDCLK); no longer C29.2 (SWDCLK)
- net SYNC: now also FPC1.4; no longer FPC1.20
- net VDD: now also C29.2 (VDD), C15.2; no longer C29.4 (VDD), C36.2
- net at R8.2: now also FPC1.5; no longer FPC1.19
- net at U7.3 (P0.01_XL2), X1.2: now also C12.1; no longer C44.1
- net at U7.28 (XC1), X2.3: now also C26.2
- net at U7.27 (DEC3): now also C22.2
- net at U7.2 (P0.00_XL1), X1.1: now also C11.1; no longer C45.1
- new net: R3.1, R4.2

Commit message: Finished routing
Connections:
- net INT_ACC2: no longer names the net of LIS2DUX1.11 (INT2)
- net INT_MAG: no longer names the net of U1.7 (INT/DRDY)
- no-connect marks 15 -> 17
Other:
- note added: "MICROCONTROLLER"
- note removed: "MCU"
- title: (none) -> DIVE COMPUTER
- moved on the sheet: ANT1, C11, C12, C13, C14, C15, C16, C17, C18, C19, C20, C21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
