File: V2/Hardware/DiveComputerV2/DiveComputerV2.kicad_pcb (KiCad board)
At the start: 4 copper layers, 36.3 x 36.3 mm, 86 parts, among them J1 Conn_01x01_Socket, J2 Conn_01x01_Socket, J3 Conn_01x02_Socket, U1 LIS2MDL, U10 MS583730BA01-50, U11 TPS7A0331PDQNR, U12 TPS75105DSKR, U2 NRF52833-QDAA-R, U3 TPS7A0218PDQNR, U4 DRV2624YFFR, U5 BQ51051BRHLR, U6 TPS7A0212PYCHR, U8 VEML6035, U9 TMAG3001A1Y, X1 ECS-320-CDX-2152, X2 CM8V-T1A-32.768KHZ-9PF-20PPM-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

Commit message: PCB layout
Parts:
- removed the C25 at (100.5, 34.5)
- removed the C27 at (100.5, 38.5)
- removed the C28 at (110.7, 65.0)
- removed the C29 at (108.0, 62.3)
- removed the C31 at (108.0, 59.8)
- removed the C39 at (103.4, 51.7)
- removed the C42 at (101.6, 51.4)
- removed the C48 at (96.0, 35.8)
- removed the C49 at (96.1, 37.6)
- added C11: 12p, Capacitor_SMD:C_0402_1005Metric, F.Cu at (100.0, 60.8)
- added C12: 12p, Capacitor_SMD:C_0402_1005Metric, F.Cu at (100.0, 62.3)
- added C14: 4.7u, Capacitor_SMD:C_0402_1005Metric, F.Cu at (108.2, 59.8)
- added C15: 1u, Capacitor_SMD:C_0402_1005Metric, F.Cu at (99.4, 59.7)
- added C22: 100p, Capacitor_SMD:C_0402_1005Metric, F.Cu at (103.4, 51.7)
- added C26: 12p, Capacitor_SMD:C_0402_1005Metric, F.Cu at (101.7, 51.4)
- added C34: 1u, Capacitor_SMD:C_0402_1005Metric, F.Cu at (96.8, 65.0)
- added C35: 1u, Capacitor_SMD:C_0402_1005Metric, F.Cu at (98.0, 63.3)
- added C43: 1u, Capacitor_SMD:C_0402_1005Metric, F.Cu at (96.8, 66.0)
- added G***: LOGO, LOGO, B.Cu at (105.3, 61.9)
- added R3: 22k, Resistor_SMD:R_0402_1005Metric, F.Cu at (109.0, 66.5)
- C2: renamed from C10; moved to B.Cu
- C44, C45: value 12p -> 1u
- R4: renamed from R10; value 26.7k -> 4.7k
- U5: renamed from U10; moved to B.Cu
- moved C2 51.9 mm to (103.8, 77.4), turned to 90 degrees
- moved U5 39.1 mm to (107.3, 76.9), turned to 90 degrees
- moved U10 32.5 mm to (96.8, 69.0), turned to -90 degrees
- moved R4 30.7 mm to (107.0, 66.6)
- moved U6 29.6 mm to (107.6, 64.6), turned to 180 degrees
- moved U8 28.8 mm to (98.6, 65.4)
- moved R7 28.8 mm to (111.0, 64.1)
- moved R8 28.7 mm to (111.0, 65.1)
- moved R6 18.2 mm to (93.5, 60.4), turned to 90 degrees
- moved R5 16.6 mm to (92.5, 60.4), turned to 90 degrees
- moved U9 12.5 mm to (97.5, 61.7), turned to 180 degrees
- moved C45 8.83 mm to (98.5, 69.5)
- moved C36 8.70 mm to (98.5, 68.3)
- moved C7 6.51 mm to (91.3, 63.6)
- moved LIS2DUX1 6.28 mm to (91.7, 65.4)
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- renumbered C4 to C1, C2 to C10, C32 to C13, C33 to C16, C37 to C17, C38 to C18, C34 to C19, C35 to C20, C50 to C21, C40 to C23, C41 to C24, C43 to C25, C46 to C27, C47 to C28, C6 to C29, C21 to C3, C18 to C31, C12 to C32, C11 to C33, C7 to C37, C8 to C38, C9 to C39, C26 to C4, C13 to C40, C14 to C41, C15 to C42, C16 to C46, C20 to C47, C17 to C48, C22 to C49, C3 to C5, C5 to C6, C1 to C7, C23 to C8, C24 to C9, L3 to L1, L4 to L3, L5 to L4, L1 to L5, LIS2DUX12 to LIS2DUX1, R9 to R1, R5 to R10, R6 to R11, R3 to R12, R4 to R13, R8 to R2, R1 to R5, R2 to R6, R12 to R7, R11 to R8, R7 to R9, U3 to U10, U5 to U11, U8 to U2, U4 to U3, U9 to U4, U12 to U6, U2 to U7, U6 to U8, U11 to U9, X2 to X1, X1 to X2
Connections:
- C29 pad 2: /SWDCLK -> VDD
- C29 pad 4: VDD -> /SWDCLK
- C36 pad 2: VDD -> +1.8V
- C44 pad 1: Net-(U2-P0.01_XL2) -> GND
- C44 pad 2: GND -> BAT+
- C45 pad 1: Net-(U2-P0.00_XL1) -> GND
- C45 pad 2: GND -> BAT+
- FPC1 pad 1: unconnected-(FPC1-Pad1) -> GND
- FPC1 pad 10: GND -> /SCREEN_~{CS}
- FPC1 pad 11: /SCREEN_SDI -> +1.8V
- FPC1 pad 13: +1.8V -> /SCREEN_SDI
- FPC1 pad 14: /SCREEN_~{CS} -> GND
- FPC1 pad 15: GND -> +1.2V
- FPC1 pad 16: /SCREEN_~{RST} -> +1.2V
- FPC1 pad 18: GND -> +1.2V
- FPC1 pad 19: Net-(FPC1-Pad19) -> +1.2V
- FPC1 pad 2: +3.1V -> /BL
- FPC1 pad 20: /SYNC -> GND
- FPC1 pad 21: unconnected-(FPC1-Pad21) -> +1.8V
- FPC1 pad 22: /BL -> +3.1V
- FPC1 pad 23: GND -> unconnected-(FPC1-Pad23)
- FPC1 pad 3: +1.8V -> unconnected-(FPC1-Pad3)
- FPC1 pad 4: GND -> /SYNC
- FPC1 pad 5: +1.2V -> Net-(FPC1-Pad5)
- FPC1 pad 6: +1.2V -> GND
- FPC1 pad 8: +1.2V -> /SCREEN_~{RST}
- FPC1 pad 9: +1.2V -> GND
- J1 pad 1: /OUT+ -> /OUT-
- J2 pad 1: /OUT- -> /OUT+
- R4 pad 2: GND -> Net-(R3-Pad1)
- R8 pad 2: Net-(FPC1-Pad19) -> Net-(FPC1-Pad5)
- U7 pad 2: Net-(U2-P0.00_XL1) -> Net-(U7-P0.00_XL1)
- U7 pad 3: Net-(U2-P0.01_XL2) -> Net-(U7-P0.01_XL2)
- X1 pad 1: Net-(U2-P0.00_XL1) -> Net-(U7-P0.00_XL1)
- X1 pad 2: Net-(U2-P0.01_XL2) -> Net-(U7-P0.01_XL2)
Routing:
- net /SDA: track 0.00 -> 89.1 mm, vias 0 -> 7
- net /SCL: track 0.00 -> 83.0 mm, vias 0 -> 7
- net /nRESET: track 0.00 -> 33.4 mm, vias 0 -> 3
- net /1.2V_EN: track 4.69 -> 28.1 mm, vias 1 -> 2
- net /SWDCLK: track 0.00 -> 22.1 mm, vias 0 -> 1
- net /SWDIO: track 0.00 -> 21.5 mm, vias 0 -> 1
- net +1.8V: track 5.84 -> 21.4 mm, vias 0 -> 11
- net +3.1V: track 4.09 -> 17.8 mm, vias 0 -> 2
- net Net-(U11-AC1): track 13.8 -> 1.00 mm
- net /3.1V_EN: track 23.2 -> 12.3 mm
- net /SYNC: track 19.4 -> 30.0 mm, vias 0 -> 2
- net VDD: track 8.02 -> 18.5 mm, vias 0 -> 4
- net /BL_PWM_MCU: track 0.00 -> 10.3 mm
- net /INT_ACC1: track 10.5 -> 20.6 mm
- net /OUT-: track 3.28 -> 13.0 mm
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- added copper zone on F.Cu, net +1.2V
- added copper zone on F.Cu, net +1.8V
- added copper zone on In2.Cu, net +1.8V
- added copper zone on F.Cu, net /BL_PWM
- added copper zone on F.Cu, net /INT_ENC
- added copper zone on B.Cu, net /OUT+
- added copper zone on B.Cu, net /OUT-
- added copper zone on In2.Cu, net BAT+
- added copper zone on In1.Cu, net GND
- added copper zone on F.Cu, net Net-(U6-ISET)
- added copper zone on F.Cu, net VDD
- added copper zone on In2.Cu, net VDD
Other:
- outline, holes or cut-outs redrawn
- board text added: "Dive Computer v2.0 Design by Bilal YOUSFI"

Commit message: Finished routing
Parts:
- moved C6 0.45 mm to (115.9, 65.7), turned to 0 degrees
- moved R2 0.15 mm to (115.9, 66.7), turned to 0 degrees
- turned C36 to 180 degrees
Connections:
- LIS2DUX1 pad 11: /INT_ACC2 -> unconnected-(LIS2DUX1-INT2-Pad11)
- U1 pad 7: /INT_MAG -> unconnected-(U1-INT/DRDY-Pad7)
Routing:
- net +3.1V: track 17.8 -> 9.71 mm
- net +1.2V: track 6.16 -> 13.5 mm
- net /SCREEN_SCL: track 10.4 -> 15.8 mm
- net VDD: track 18.5 -> 16.5 mm
- net +1.8V: track 21.4 -> 23.2 mm
- net /INT_ENC: track 30.9 -> 31.5 mm
- net BAT+: track 9.71 -> 10.3 mm, vias 8 -> 9
- net GND: vias 216 -> 213

Commit message: LVGL Simulator
created an LVGL simulator for UID dev
Parts:
- moved R3 0.82 mm to (109.8, 66.4)
- moved R4 0.82 mm to (107.8, 66.4)
- moved R8 0.82 mm to (111.8, 64.9)
- moved U6 0.82 mm to (108.4, 64.5)
- moved R7 0.82 mm to (111.8, 64.0)
Routing:
- net /SCREEN_SCL: track 15.8 -> 25.7 mm
- net Net-(FPC1-Pad5): track 8.25 -> 9.94 mm
- net BAT+: track 10.3 -> 9.71 mm, vias 9 -> 8
- net GND: vias 213 -> 201
Other:
- outline, holes or cut-outs redrawn
